Commit message: Renaming

File: defs/pioneer3dx.xacro (robot description, xacro)
@@ -1,4 +1,4 @@
 <?xml version="1.0"?>
 <robot name="pioneer3dx" xmlns:xacro="http://ros.org/wiki/xacro">
-  <xacro:include filename="$(find pioneer3dx_cartographer)/defs/pioneer3dx_body.xacro"/>
+  <xacro:include filename="$(find pioneer3dx_explorer)/defs/pioneer3dx_body.xacro"/>
 </robot>

File: defs/pioneer3dx_body.xacro (robot description, xacro)
@@ -1,5 +1,5 @@
 <?xml version="1.0"?>
 <robot xmlns:xacro="http://ros.org/wiki/xacro">
-  <xacro:include filename="$(find pioneer3dx_cartographer)/defs/pioneer3dx_wheel.xacro"/>
+  <xacro:include filename="$(find pioneer3dx_explorer)/defs/pioneer3dx_wheel.xacro"/>
   <!-- Chassis description -->
   <link name="base_link">
@@ -16,5 +16,5 @@
 	  <origin xyz="-0.045 0 0.148" rpy="0 0 0"/>
 	  <geometry name="pioneer_geom">
-		<mesh filename="package://pioneer3dx_cartographer/meshes/chassis.stl"/>
+		<mesh filename="package://pioneer3dx_explorer/meshes/chassis.stl"/>
 	  </geometry>
 	  <material name="ChassisRed">
@@ -45,5 +45,5 @@
 	  <origin xyz="0 0 0" rpy="0 0 0"/>
 	  <geometry name="pioneer_geom">
-		<mesh filename="package://pioneer3dx_cartographer/meshes/top.stl"/>
+		<mesh filename="package://pioneer3dx_explorer/meshes/top.stl"/>
 	  </geometry>
 	  <material name="TopBlack">
@@ -71,5 +71,5 @@
 	  <origin xyz="0 0 0" rpy="0 0 0"/>
 	  <geometry name="pioneer_geom">
-		<mesh filename="package://pioneer3dx_cartographer/meshes/swivel.stl"/>
+		<mesh filename="package://pioneer3dx_explorer/meshes/swivel.stl"/>
 	  </geometry>
 	  <material name="swivel">
@@ -100,5 +100,5 @@
 	  <origin xyz="0 0 0" rpy="0 0 0"/>
 	  <geometry name="pioneer_geom">
-		<mesh filename="package://pioneer3dx_cartographer/meshes/center_hubcap.stl"/>
+		<mesh filename="package://pioneer3dx_explorer/meshes/center_hubcap.stl"/>
 	  </geometry>
 	  <material name="swivel">
@@ -129,5 +129,5 @@
 	  <origin xyz="0 0 0" rpy="0 0 0"/>
 	  <geometry name="pioneer_geom">
-		<mesh filename="package://pioneer3dx_cartographer/meshes/center_wheel.stl"/>
+		<mesh filename="package://pioneer3dx_explorer/meshes/center_wheel.stl"/>
 	  </geometry>
 	  <material name="WheelBlack">
@@ -138,5 +138,5 @@
 	  <origin xyz="0 0 0" rpy="${-3.1415927/2.0} 0 0"/>
 	  <geometry>
-		<!--<mesh filename="package://pioneer3dx_cartographer/meshes/center_wheel.stl"/>-->
+		<!--<mesh filename="package://pioneer3dx_explorer/meshes/center_wheel.stl"/>-->
 		<cylinder radius="0.0375" length="0.0314"/>
 	  </geometry>
@@ -164,5 +164,5 @@
 	  <origin xyz="0 0 0" rpy="0 0 0"/>
 	  <geometry name="pioneer_geom">
-		<mesh filename="package://pioneer3dx_cartographer/meshes/front_sonar.stl"/>
+		<mesh filename="package://pioneer3dx_explorer/meshes/front_sonar.stl"/>
 	  </geometry>
 	  <material name="SonarYellow">
@@ -189,5 +189,5 @@
 	  <origin xyz="0 0 0" rpy="0 0 0"/>
 	  <geometry name="pioneer_geom">
-		<mesh filename="package://pioneer3dx_cartographer/meshes/back_sonar.stl"/>
+		<mesh filename="package://pioneer3dx_explorer/meshes/back_sonar.stl"/>
 	  </geometry>
 	  <material name="SonarYellow">

File: defs/pioneer3dx_wheel.xacro (robot description, xacro)
@@ -1,5 +1,5 @@
 <?xml version="1.0"?>
 <robot xmlns:xacro="http://ros.org/wiki/xacro">
-  <xacro:include filename="$(find pioneer3dx_cartographer)/defs/materials.xacro"/>
+  <xacro:include filename="$(find pioneer3dx_explorer)/defs/materials.xacro"/>
   <!-- Properties (Constants) -->
   <xacro:property name="M_PI" value="3.14159"/>
@@ -16,5 +16,5 @@
         <origin xyz="0 0 0" rpy="0 0 0"/>
         <geometry name="pioneer_geom">
-          <mesh filename="package://pioneer3dx_cartographer/meshes/${suffix}_wheel.stl"/>
+          <mesh filename="package://pioneer3dx_explorer/meshes/${suffix}_wheel.stl"/>
         </geometry>
         <material name="WheelBlack">
@@ -44,5 +44,5 @@
         <origin xyz="0 0 0" rpy="0 0 0"/>
         <geometry name="pioneer_geom">
-          <mesh filename="package://pioneer3dx_cartographer/meshes/${suffix}_hubcap.stl"/>
+          <mesh filename="package://pioneer3dx_explorer/meshes/${suffix}_hubcap.stl"/>
         </geometry>
         <material name="HubcapYellow">
