Commit message: Reorganize folders to integrate more algorithms

File: defs/pioneer3dx_body.xacro (robot description, xacro)
@@ -60,4 +60,26 @@
 	<child link="top_plate"/>
   </joint>
+    <joint name="laser_joint" type="fixed">
+    <parent link="top_plate"/>
+    <child link="laser_link"/>
+    <origin rpy="0 0 0" xyz="0.12 0 0.07"/>
+  </joint>
+  <link name="laser_link">
+    <visual>
+      <geometry>
+        <mesh filename="package://pioneer3dx_explorer/meshes/laser.stl"/>
+      </geometry>
+      <material name="blue">
+        <color rgba="0.24 0.63 0.86 1"/>
+      </material>
+    </visual>
+  </link>
+  <joint name="imu_joint" type="fixed">
+    <parent link="top_plate"/>
+    <child link="imu_link"/>
+    <origin rpy="0 0 0" xyz="-0.038 0 0.112"/>
+  </joint>
+  <link name="imu_link">
+  </link>
   <!-- Swivel -->
   <link name="swivel">
@@ -151,6 +173,6 @@
 	<child link="center_hubcap"/>
   </joint>
-  <xacro:p3dx_wheel suffix="left" parent="base_link" reflect="1"/>
-  <xacro:p3dx_wheel suffix="right" parent="base_link" reflect="-1"/>
+  <xacro:p3dx_wheel suffix="left" parent="base_link" reflect="1.0"/>
+  <xacro:p3dx_wheel suffix="right" parent="base_link" reflect="-1.0"/>
   <!-- Front + Back Sonar -->
   <link name="front_sonar">

File: defs/pioneer3dx_wheel.xacro (robot description, xacro)
@@ -1,7 +1,5 @@
 <?xml version="1.0"?>
 <robot xmlns:xacro="http://ros.org/wiki/xacro">
-  <xacro:include filename="$(find pioneer3dx_explorer)/defs/materials.xacro"/>
-  <!-- Properties (Constants) -->
-  <xacro:property name="M_PI" value="3.14159"/>
+  <xacro:include filename="materials.xacro"/>
   <!-- Right/Left Hubcap + Wheel -->
   <xacro:macro name="p3dx_wheel" params="suffix parent reflect">
@@ -52,9 +50,9 @@
     </link>
     <!-- The transmission tag is used only by ros_control -->
-    <!--<transmission type="pr2_mechanism_model/SimpleTransmission" name="${parent}_${suffix}_wheel_trans">
+    <transmission type="pr2_mechanism_model/SimpleTransmission" name="${parent}_${suffix}_wheel_trans">
         <actuator name="base_${suffix}_wheel_motor" />
         <joint name="base_${suffix}_wheel_joint" />
         <mechanicalReduction>${reflect * 624/35 * 80/19}</mechanicalReduction>
-        </transmission>-->
+        </transmission>
     <joint name="base_${suffix}_wheel_joint" type="continuous">
       <axis xyz="0 1 0"/>
